File: kicad-pcb/microvan.sch (KiCad schematic (older format))
At the start: 89 parts, among them U1 ProMicro

Commit message: Fix routing and add edge cuts.
Parts:
- D1, D10, D11, D12, D13, D14, D15, D16, D17, D18, D19, D2, D20, D21, D22, D23, D24, D25, D26, D27, D28, D29, D3, D30, D31, D32, D33, D34, D35, D36, D37, D38, D39, D4, D40, D41, D42, D43, D44, D5, D6, D7, D8, D9: footprint (none) -> Keebio-Parts:Diode-Hybrid-Back
- MX1, MX10, MX11, MX14, MX15, MX16, MX17, MX18, MX19, MX2, MX20, MX21, MX22, MX23, MX26, MX27, MX28, MX29, MX3, MX30, MX31, MX32, MX33, MX34, MX35, MX36, MX4, MX5, MX6, MX7, MX8, MX9: footprint (none) -> MX_Alps_Hybrid:MX-1U-NoLED
- MX12, MX25, MX44: footprint (none) -> MX_Alps_Hybrid:MX-1.75U-NoLED
- MX13, MX37, MX39, MX42: footprint (none) -> MX_Alps_Hybrid:MX-1.25U-NoLED
- MX24, MX38, MX43: footprint (none) -> MX_Alps_Hybrid:MX-1.5U-NoLED
- MX40: footprint (none) -> MX_Alps_Hybrid:MX-2.25U-ReversedStabilizers-NoLED
- MX41: footprint (none) -> MX_Alps_Hybrid:MX-2U-ReversedStabilizers-NoLED
- U1: footprint (none) -> Keebio-Parts:ArduinoProMicro-BackSide
Connections:
- net COL12 is gone; now on net COL11: MX12.1 (COL), MX24.1 (COL), MX36.1 (COL)
- net COL0: now also U1.7 (4/PD4)
- net COL1: now also MX26.1 (COL), MX38.1 (COL), U1.8 (5/PC6)
- net COL10: now also MX35.1 (COL), MX44.1 (COL), U1.17 (A0/PF7)
- net COL11: now also U1.6 (3/PD0); no longer MX35.1 (COL), MX44.1 (COL)
- net COL2: now also MX27.1 (COL), MX39.1 (COL), U1.9 (6/PD7)
- net COL3: now also MX28.1 (COL), U1.10 (7/PE6)
- net COL4: now also MX17.1 (COL), MX29.1 (COL), MX40.1 (COL), MX5.1 (COL), U1.11 (8/PB4)
- net COL5: now also MX30.1 (COL), U1.12 (9/PB5)
- net COL6: now also MX31.1 (COL), MX41.1 (COL), U1.13 (10/PB6)
- net COL7: now also MX32.1 (COL), MX42.1 (COL), U1.14 (16/PB2)
- net COL8: now also MX33.1 (COL), U1.15 (14/PB3)
- net COL9: now also MX34.1 (COL), MX43.1 (COL), U1.16 (15/PB1)
- net ROW0: now also U1.5 (2/PD1)
- net ROW1: now also U1.18 (A1/PF6); no longer MX26.1 (COL), MX27.1 (COL), MX28.1 (COL), MX29.1 (COL), MX30.1 (COL), MX31.1 (COL), MX32.1 (COL), MX33.1 (COL), MX34.1 (COL), MX38.1 (COL), MX39.1 (COL), MX40.1 (COL), MX41.1 (COL), MX42.1 (COL), MX43.1 (COL)
- net ROW2: now also U1.19 (A2/PF5)
- net ROW3: now also U1.20 (A3/PF4)
