File: kicad-pcb/microvan.kicad_pcb (KiCad board)
At the start: 2 copper layers, 241.3 x 74.6 mm, 90 parts, among them U1 ProMicro

Commit message: Add mounting holes
Parts:
- added .: MountingHole_2.5mm, MountingHole:MountingHole_2.5mm, F.Cu at (144.5, 114.3)
- added REF**: MountingHole_2.5mm, MountingHole:MountingHole_2.5mm, F.Cu at (77.8, 133.3)
- added REF**: MountingHole_2.5mm, MountingHole:MountingHole_2.5mm, F.Cu at (77.8, 95.2)
- added REF**: MountingHole_2.5mm, MountingHole:MountingHole_2.5mm, F.Cu at (215.9, 95.2)
- added REF**: MountingHole_2.5mm, MountingHole:MountingHole_2.5mm, F.Cu at (215.9, 133.3)
Routing:
- net COL9: track 92.0 -> 96.4 mm
- net COL5: track 151.1 -> 153.5 mm
- net COL4: track 191.4 -> 193.7 mm
